Commit message: The sim is ready w/o sensors now i want to learn how to control it via python

File: dev_ws/src/balance_bot/description/robot.urdf.xacro (robot description, xacro)
@@ -2,3 +2,4 @@
 <robot xmlns:xacro="http://www.ros.org/wiki/xacro"  name="balance_bot">
     <xacro:include filename="robot_core.xacro" />
+    <!-- <xacro:include filename="gazebo_control.xacro" /> -->
 </robot>

File: dev_ws/src/balance_bot/description/robot_core.xacro (robot description, xacro)
@@ -21,5 +21,5 @@
     <parent link="base_link"/>
     <child link="chassis"/>
-    <origin xyz="0 0 0"/>
+    <origin xyz="0 0 0.1"/>
 </joint>
 <link name ="chassis">
@@ -41,9 +41,12 @@
     </xacro:inertial_box>
 </link>
+<gazebo refrence="chassis">
+    <material>Gazebo/white</material>
+</gazebo>
 <!-- right wheel -->
 <joint name ="right_wheel_joint" type="continuous">
     <parent link="base_link"/>
     <child link="right_wheel"/>
-    <origin xyz="0 -0.1 0" rpy="${pi/2} 0 0"/>
+    <origin xyz="0 -0.1 0.1" rpy="${pi/2} 0 0"/>
     <axis xyz="0 0 -1"></axis>
 </joint>
@@ -64,9 +67,12 @@
     </xacro:inertial_cylinder>
 </link>
+<gazebo refrence="right_wheel">
+    <material>Gazebo/blue</material>
+</gazebo>
 <!-- left wheel -->
 <joint name ="left_wheel_joint" type="continuous">
     <parent link="base_link"/>
     <child link="left_wheel"/>
-    <origin xyz="0 0.1 0" rpy="-${pi/2} 0 0"/>
+    <origin xyz="0 0.1 0.1" rpy="-${pi/2} 0 0"/>
     <axis xyz="0 0 1"></axis>
 </joint>
@@ -87,3 +93,6 @@
     </xacro:inertial_cylinder>
 </link>
+<gazebo refrence="left_wheel">
+    <material>Gazebo/blue</material>
+</gazebo>
 </robot>
