Commit message: Robot not moving but save checkpoint

File: dev_ws/src/balance_bot/description/gazebo_control.xacro (robot description, xacro)
@@ -11,4 +11,5 @@
             <max_wheel_torque>200</max_wheel_torque>
             <max_wheel_acceleration>10.0</max_wheel_acceleration>
+            <command_topic>cmd_vel</command_topic>
             <!-- Output -->
             <odometry_frame>odom</odometry_frame>

File: dev_ws/src/balance_bot/description/robot.urdf.xacro (robot description, xacro)
@@ -2,4 +2,5 @@
 <robot xmlns:xacro="http://www.ros.org/wiki/xacro"  name="balance_bot">
     <xacro:include filename="robot_core.xacro" />
+    <xacro:include filename="ros2_control.xacro" />
     <!-- <xacro:include filename="gazebo_control.xacro" /> -->
 </robot>

File: dev_ws/src/balance_bot/description/robot_core.xacro (robot description, xacro)
@@ -48,5 +48,5 @@
     <parent link="base_link"/>
     <child link="right_wheel"/>
-    <origin xyz="0 -0.1 0.1" rpy="${pi/2} 0 0"/>
+    <origin xyz="0 -0.125 0.1" rpy="${pi/2} 0 0"/>
     <axis xyz="0 0 -1"></axis>
 </joint>
@@ -54,5 +54,5 @@
     <visual>
         <geometry>
-            <cylinder radius="0.1" length="0.04"/>
+            <cylinder radius="0.1" length="0.05"/>
         </geometry>
         <material name="blue"/>
@@ -60,8 +60,15 @@
     <collision>
         <geometry>
-            <cylinder radius="0.1" length="0.04"/>
+            <cylinder radius="0.1" length="0.05"/>
         </geometry>
+        <surface>
+            <friction>
+                <ode>
+                    <mu>1.0</mu>      <mu2>1.0</mu2>
+                </ode>
+            </friction>
+        </surface>
     </collision>
-    <xacro:inertial_cylinder mass="0.1" length="0.04" radius="0.1">
+    <xacro:inertial_cylinder mass="0.1" length="0.05" radius="0.1">
         <origin xyz="0 0 0" rpy="0 0 0"/>
     </xacro:inertial_cylinder>
@@ -74,5 +81,5 @@
     <parent link="base_link"/>
     <child link="left_wheel"/>
-    <origin xyz="0 0.1 0.1" rpy="-${pi/2} 0 0"/>
+    <origin xyz="0 0.125 0.1" rpy="-${pi/2} 0 0"/>
     <axis xyz="0 0 1"></axis>
 </joint>
@@ -80,5 +87,5 @@
     <visual>
         <geometry>
-            <cylinder radius="0.1" length="0.04"/>
+            <cylinder radius="0.1" length="0.05"/>
         </geometry>
         <material name="blue"/>
@@ -86,8 +93,15 @@
     <collision>
         <geometry>
-            <cylinder radius="0.1" length="0.04"/>
+            <cylinder radius="0.1" length="0.05"/>
         </geometry>
+        <surface>
+            <friction>
+                <ode>
+                    <mu>1.0</mu>      <mu2>1.0</mu2>
+                </ode>
+            </friction>
+        </surface>
     </collision>
-    <xacro:inertial_cylinder mass="0.1" length="0.04" radius="0.1">
+    <xacro:inertial_cylinder mass="0.1" length="0.05" radius="0.1">
         <origin xyz="0 0 0" rpy="0 0 0"/>
     </xacro:inertial_cylinder>
